File: PitayaGoAdapter.kicad_pcb (KiCad board)
At the start: 2 copper layers, 56.1 x 25.5 mm, 2 parts, among them J1 Conn_01x14, J2 Conn_01x14

Commit message: Update sch and pcb
Signed-off-by: DevriesL <therkduan@gmail.com>
Parts:
- added C1: 47pF, Capacitor_SMD:C_0402_1005Metric, F.Cu at (120.6, 23.1)
- added C12: 47pF, Capacitor_SMD:C_0402_1005Metric, F.Cu at (124.8, 19.1)
- added C2: 47pF, Capacitor_SMD:C_0402_1005Metric, F.Cu at (123.5, 21.1)
- added C51: 1uF, Capacitor_SMD:C_0603_1608Metric, F.Cu at (90.7, 31.9)
- added C52: 1uF, Capacitor_SMD:C_0603_1608Metric, F.Cu at (94.7, 31.9)
- added J3: HAPTIC_Conn, Connector_JST:JST_PH_S2B-PH-SM4-TB_1x02-1MP_P2.00mm_Horizontal, F.Cu at (113.4, 58.0)
- added J4: HMI_Conn_0_2, Connector_JST:JST_PH_B4B-PH-SM4-TB_1x04-1MP_P2.00mm_Vertical, F.Cu at (111.4, 42.7)
- added J5: HMI_Conn_3_5, Connector_JST:JST_PH_B4B-PH-SM4-TB_1x04-1MP_P2.00mm_Vertical, F.Cu at (96.3, 42.7)
- added J6: HMI_Conn_6_8, Connector_JST:JST_PH_B4B-PH-SM4-TB_1x04-1MP_P2.00mm_Vertical, F.Cu at (61.8, 58.4)
- added R1: 10K, Resistor_SMD:R_0402_1005Metric, F.Cu at (98.1, 31.7)
- added R10: 24K, Resistor_SMD:R_0402_1005Metric, F.Cu at (117.7, 24.1)
- added R11: 24K, Resistor_SMD:R_0402_1005Metric, F.Cu at (121.9, 19.1)
- added R12: 24K, Resistor_SMD:R_0402_1005Metric, F.Cu at (124.8, 17.1)
- added R2: 10K, Resistor_SMD:R_0402_1005Metric, F.Cu at (101.0, 31.7)
- added R3: 10K, Resistor_SMD:R_0402_1005Metric, F.Cu at (119.0, 17.1)
- added R4: 0R, Resistor_SMD:R_0402_1005Metric, F.Cu at (114.8, 22.1)
- added R5: 0R, Resistor_SMD:R_0402_1005Metric, F.Cu at (114.8, 24.1)
- added R51: 2.2K, Resistor_SMD:R_0402_1005Metric, F.Cu at (120.6, 21.1)
- added R52: 2.2K, Resistor_SMD:R_0402_1005Metric, F.Cu at (114.8, 28.1)
- added R53: 10K, Resistor_SMD:R_0402_1005Metric, F.Cu at (117.7, 26.1)
- added R6: 0R, Resistor_SMD:R_0402_1005Metric, F.Cu at (119.0, 19.1)
- added R7: 4.3K, Resistor_SMD:R_0402_1005Metric, F.Cu at (121.9, 17.1)
- added R8: 4.3K, Resistor_SMD:R_0402_1005Metric, F.Cu at (117.7, 22.1)
- added R9: 4.3K, Resistor_SMD:R_0402_1005Metric, F.Cu at (114.8, 26.1)
- added U3: DRV2605LDGS, Package_SO:VSSOP-10_3x3mm_P0.5mm, F.Cu at (98.9, 54.6)
Connections:
- net Net-(J1-Pad10) renamed /P0.29
- net Net-(J1-Pad11) renamed /P0.28
- net Net-(J1-Pad3) renamed /RESET
- net Net-(J1-Pad4) renamed /SWCLK
- net Net-(J1-Pad5) renamed /SWDIO
- net Net-(J1-Pad8) renamed /P0.31
- net Net-(J1-Pad9) renamed /P0.30
- net Net-(J2-Pad1) renamed /P0.25
- net Net-(J2-Pad10) renamed /P0.14
- net Net-(J2-Pad11) renamed /P0.13
- net Net-(J2-Pad14) renamed /MB_VIN
- net Net-(J2-Pad2) renamed /P0.24
- net Net-(J2-Pad3) renamed /P0.23
- net Net-(J2-Pad4) renamed /P0.22
- net Net-(J2-Pad5) renamed /P0.21
- net Net-(J2-Pad6) renamed /P0.20
- net Net-(J2-Pad7) renamed /P0.17
- net Net-(J2-Pad8) renamed /P0.16
- net Net-(J2-Pad9) renamed /P0.15
- J1 pad 1: Net-(J1-Pad1) -> /MB_3V3
- J1 pad 12: Net-(J1-Pad12) -> /P0.05
- J1 pad 13: Net-(J1-Pad13) -> /P0.04
- J1 pad 14: Net-(J1-Pad14) -> /P0.03
- J1 pad 2: Net-(J1-Pad2) -> GND
- J1 pad 6: Net-(J1-Pad6) -> /P0.27
- J1 pad 7: Net-(J1-Pad7) -> /P0.26
- J2 pad 12: Net-(J2-Pad12) -> GND
- J2 pad 13: Net-(J2-Pad13) -> /MB_4V4
Other:
- board size 56.1 x 25.5 mm -> 67.1 x 25.5 mm
